File: PCB/hotswap_choc/helixhschoc.sch (KiCad schematic (older format))
At the start: 126 parts, among them J1 MJ-4PP-9, P1 CONN_01X01, P2 CONN_01X01, P3 OLED, P4 LED, SW1 SW_PUSH, SW10 SW_PUSH, SW11 SW_PUSH, SW12 SW_PUSH, SW13 SW_PUSH, SW14 SW_PUSH, SW15 SW_PUSH, SW16 SW_PUSH, SW17 SW_PUSH, SW18 SW_PUSH, SW19 SW_PUSH, SW2 SW_PUSH, SW20 SW_PUSH, SW21 SW_PUSH, SW22 SW_PUSH, SW23 SW_PUSH, SW24 SW_PUSH, SW25 SW_PUSH, SW26 SW_PUSH, SW27 SW_PUSH, SW28 SW_PUSH, SW29 SW_PUSH, SW3 SW_PUSH, SW30 SW_PUSH, SW31 SW_PUSH, SW32 SW_PUSH, SW33 Reset, SW4 SW_PUSH, SW5 SW_PUSH, SW6 SW_PUSH, SW7 SW_PUSH, SW8 SW_PUSH, SW9 SW_PUSH, U1 ProMicro, U10 SK6812mini, U11 SK6812mini, U12 SK6812mini, U13 SK6812mini, U14 SK6812mini, U15 SK6812mini, U16 SK6812mini, U17 SK6812mini, U18 SK6812mini, U19 SK6812mini, U2 SK6812mini, U20 SK6812mini, U21 SK6812mini, U22 SK6812mini, U23 SK6812mini, U24 SK6812mini, U25 SK6812mini, U26 SK6812mini, U27 SK6812mini, U28 SK6812mini, U29 SK6812mini, U3 SK6812mini, U30 SK6812mini, U31 SK6812mini, U32 SK6812mini, U33 SK6812mini, U4 SK6812mini, U5 SK6812mini, U6 SK6812mini, U7 SK6812mini, U8 SK6812mini, U9 SK6812mini

Commit message: PCB WIP
Parts:
- JP10, JP11, JP4, JP5, JP7, JP8, JP9: symbol helixhschoc-rescue:JP2 -> random-keyboard-parts:Jumper_Small
- SW33: footprint MYLIB:SW_3.5x6.0_TH -> Random-keyboard-parts:SW_3.5x6.0_TH
- U10, U11, U12, U13, U14, U15, U16, U17, U18, U19, U20, U21, U22, U23, U24, U25, U26, U27, U28, U29, U3, U30, U31, U32, U33, U4, U5, U6, U7, U8, U9: footprint MYLIB_REV:SK6812MINI_rev -> LED_WS_SK:SK6812MINI_rev
- U2: footprint JMG:SK6812MINI_rev -> LED_WS_SK:SK6812MINI_rev

Commit message: Pcb update
Parts:
- H1, H2, H3, H4, H5, H6, H7, H8, H9: footprint JMG:HOLE_M2_TH -> Random-keyboard-parts:HOLE_M2_TH
- H10, H11, H12, H13: footprint JMG:HOLE_M2 -> Random-keyboard-parts:HOLE_M2
- JP10, JP11, JP4, JP5, JP6, JP7, JP8, JP9: footprint MYLIB:Jumper -> Random-keyboard-parts:Jumper_Small
- P1, P2: footprint MYLIB:1PIN_0.1 -> Random-keyboard-parts:Pin_Small
- P3: footprint MYLIB:MY_SIL-4 -> Random-keyboard-parts:OLED_Small
- P4: footprint MYLIB_REV:StripLED_rev -> Random-keyboard-parts:LED_Strip_Pad
Changed lines of the file:
@@
 F 0 "P3" H 2600 5100 50  0000 C CNN
 F 1 "OLED" V 2700 4850 50  0000 C CNN
-F 2 "MYLIB:MY_SIL-4" H 2600 4850 50  0001 C CNN
+F 2 "Random-keyboard-parts:OLED_Small" H 2600 4850 50  0001 C CNN
 F 3 "" H 2600 4850 50  0000 C CNN
 	1    2600 4850
@@
 F 0 "P4" H 6600 5050 50  0000 C CNN
 F 1 "LED" V 6700 4850 50  0000 C CNN
-F 2 "MYLIB_REV:StripLED_rev" H 6600 4850 50  0001 C CNN
+F 2 "Random-keyboard-parts:LED_Strip_Pad" H 6600 4850 50  0001 C CNN
 F 3 "" H 6600 4850 50  0000 C CNN
 	1    6600 4850
@@
 F 0 "P1" V 6200 3150 50  0000 C CNN
 F 1 "CONN_01X01" V 6200 3150 50  0001 C CNN
-F 2 "MYLIB:1PIN_0.1" H 6100 3150 50  0001 C CNN
+F 2 "Random-keyboard-parts:Pin_Small" H 6100 3150 50  0001 C CNN
 F 3 "" H 6100 3150 50  0000 C CNN
 	1    6100 3150
@@
 F 0 "P2" V 6200 2300 50  0000 C CNN
 F 1 "CONN_01X01" V 6200 2300 50  0001 C CNN
-F 2 "MYLIB:1PIN_0.1" H 6100 2300 50  0001 C CNN
+F 2 "Random-keyboard-parts:Pin_Small" H 6100 2300 50  0001 C CNN
 F 3 "" H 6100 2300 50  0000 C CNN
 	1    6100 2300
@@
 F 0 "JP5" V 3500 4900 50  0000 C CNN
 F 1 "VCC" H 3500 4751 40  0001 C CNN
-F 2 "MYLIB:Jumper" H 3400 4900 60  0001 C CNN
+F 2 "Random-keyboard-parts:Jumper_Small" H 3400 4900 60  0001 C CNN
 F 3 "" H 3400 4900 60  0000 C CNN
 	1    3400 4900
@@
 F 0 "JP6" V 3500 5100 50  0000 C CNN
 F 1 "SCL" H 3500 4951 40  0001 C CNN
-F 2 "MYLIB:Jumper" H 3400 5100 60  0001 C CNN
+F 2 "Random-keyboard-parts:Jumper_Small" H 3400 5100 60  0001 C CNN
 F 3 "" H 3400 5100 60  0000 C CNN
 	1    3400 5100
@@
 F 0 "JP7" V 3500 5300 50  0000 C CNN
 F 1 "SDA" H 3500 5151 40  0001 C CNN
-F 2 "MYLIB:Jumper" H 3400 5300 60  0001 C CNN
+F 2 "Random-keyboard-parts:Jumper_Small" H 3400 5300 60  0001 C CNN
 F 3 "" H 3400 5300 60  0000 C CNN
 	1    3400 5300
@@
 F 0 "JP8" V 3500 5800 50  0000 C CNN
 F 1 "SDA" H 3500 5651 40  0001 C CNN
-F 2 "MYLIB:Jumper" H 3400 5800 60  0001 C CNN
+F 2 "Random-keyboard-parts:Jumper_Small" H 3400 5800 60  0001 C CNN
 F 3 "" H 3400 5800 60  0000 C CNN
 	1    3400 5800
@@
 F 0 "JP9" V 3500 6000 50  0000 C CNN
 F 1 "SCL" H 3500 5851 40  0001 C CNN
-F 2 "MYLIB:Jumper" H 3400 6000 60  0001 C CNN
+F 2 "Random-keyboard-parts:Jumper_Small" H 3400 6000 60  0001 C CNN
 F 3 "" H 3400 6000 60  0000 C CNN
 	1    3400 6000
@@
 F 0 "JP10" V 3500 6200 50  0000 C CNN
 F 1 "VCC" H 3500 6051 40  0001 C CNN
-F 2 "MYLIB:Jumper" H 3400 6200 60  0001 C CNN
+F 2 "Random-keyboard-parts:Jumper_Small" H 3400 6200 60  0001 C CNN
 F 3 "" H 3400 6200 60  0000 C CNN
 	1    3400 6200
@@
 F 0 "JP11" V 3500 6400 50  0000 C CNN
 F 1 "GND" H 3500 6251 40  0001 C CNN
-F 2 "MYLIB:Jumper" H 3400 6400 60  0001 C CNN
+F 2 "Random-keyboard-parts:Jumper_Small" H 3400 6400 60  0001 C CNN
 F 3 "" H 3400 6400 60  0000 C CNN
 	1    3400 6400
@@
 F 0 "H2" H 6150 6346 50  0000 L CNN
 F 1 "MountingHole" H 6150 6255 50  0000 L CNN
-F 2 "JMG:HOLE_M2_TH" H 6050 6300 50  0001 C CNN
+F 2 "Random-keyboard-parts:HOLE_M2_TH" H 6050 6300 50  0001 C CNN
 F 3 "~" H 6050 6300 50  0001 C CNN
 	1    6050 6300
@@
 F 0 "H1" H 6150 6546 50  0000 L CNN
 F 1 "MountingHole" H 6150 6455 50  0000 L CNN
-F 2 "JMG:HOLE_M2_TH" H 6050 6500 50  0001 C CNN
+F 2 "Random-keyboard-parts:HOLE_M2_TH" H 6050 6500 50  0001 C CNN
 F 3 "~" H 6050 6500 50  0001 C CNN
 	1    6050 6500
@@
 F 0 "H3" H 6150 6746 50  0000 L CNN
 F 1 "MountingHole" H 6150 6655 50  0000 L CNN
-F 2 "JMG:HOLE_M2_TH" H 6050 6700 50  0001 C CNN
+F 2 "Random-keyboard-parts:HOLE_M2_TH" H 6050 6700 50  0001 C CNN
 F 3 "~" H 6050 6700 50  0001 C CNN
 	1    6050 6700
@@
 F 0 "H4" H 6150 6946 50  0000 L CNN
 F 1 "MountingHole" H 6150 6855 50  0000 L CNN
-F 2 "JMG:HOLE_M2_TH" H 6050 6900 50  0001 C CNN
+F 2 "Random-keyboard-parts:HOLE_M2_TH" H 6050 6900 50  0001 C CNN
 F 3 "~" H 6050 6900 50  0001 C CNN
 	1    6050 6900
@@
 F 0 "H5" H 6850 6296 50  0000 L CNN
 F 1 "MountingHole" H 6850 6205 50  0000 L CNN
-F 2 "JMG:HOLE_M2_TH" H 6750 6250 50  0001 C CNN
+F 2 "Random-keyboard-parts:HOLE_M2_TH" H 6750 6250 50  0001 C CNN
 F 3 "~" H 6750 6250 50  0001 C CNN
 	1    6750 6250
@@
 F 0 "H6" H 6850 6496 50  0000 L CNN
 F 1 "MountingHole" H 6850 6405 50  0000 L CNN
-F 2 "JMG:HOLE_M2_TH" H 6750 6450 50  0001 C CNN
+F 2 "Random-keyboard-parts:HOLE_M2_TH" H 6750 6450 50  0001 C CNN
 F 3 "~" H 6750 6450 50  0001 C CNN
 	1    6750 6450
@@
 F 0 "H7" H 6850 6696 50  0000 L CNN
 F 1 "MountingHole" H 6850 6605 50  0000 L CNN
-F 2 "JMG:HOLE_M2_TH" H 6750 6650 50  0001 C CNN
+F 2 "Random-keyboard-parts:HOLE_M2_TH" H 6750 6650 50  0001 C CNN
 F 3 "~" H 6750 6650 50  0001 C CNN
 	1    6750 6650
@@
 F 0 "H8" H 6850 6896 50  0000 L CNN
 F 1 "MountingHole" H 6850 6805 50  0000 L CNN
-F 2 "JMG:HOLE_M2_TH" H 6750 6850 50  0001 C CNN
+F 2 "Random-keyboard-parts:HOLE_M2_TH" H 6750 6850 50  0001 C CNN
 F 3 "~" H 6750 6850 50  0001 C CNN
 	1    6750 6850
@@
 F 0 "H9" H 6850 7096 50  0000 L CNN
 F 1 "MountingHole" H 6850 7005 50  0000 L CNN
-F 2 "JMG:HOLE_M2_TH" H 6750 7050 50  0001 C CNN
+F 2 "Random-keyboard-parts:HOLE_M2_TH" H 6750 7050 50  0001 C CNN
 F 3 "~" H 6750 7050 50  0001 C CNN
 	1    6750 7050
@@
 F 0 "H10" H 6150 7446 50  0000 L CNN
 F 1 "MountingHole" H 6150 7355 50  0000 L CNN
-F 2 "JMG:HOLE_M2" H 6050 7400 50  0001 C CNN
+F 2 "Random-keyboard-parts:HOLE_M2" H 6050 7400 50  0001 C CNN
 F 3 "~" H 6050 7400 50  0001 C CNN
 	1    6050 7400
@@
 F 0 "H12" H 6850 7446 50  0000 L CNN
 F 1 "MountingHole" H 6850 7355 50  0000 L CNN
-F 2 "JMG:HOLE_M2" H 6750 7400 50  0001 C CNN
+F 2 "Random-keyboard-parts:HOLE_M2" H 6750 7400 50  0001 C CNN
 F 3 "~" H 6750 7400 50  0001 C CNN
 	1    6750 7400
@@
 F 0 "H11" H 6150 7646 50  0000 L CNN
 F 1 "MountingHole" H 6150 7555 50  0000 L CNN
-F 2 "JMG:HOLE_M2" H 6050 7600 50  0001 C CNN
+F 2 "Random-keyboard-parts:HOLE_M2" H 6050 7600 50  0001 C CNN
 F 3 "~" H 6050 7600 50  0001 C CNN
 	1    6050 7600
@@
 F 0 "H13" H 6850 7646 50  0000 L CNN
 F 1 "MountingHole" H 6850 7555 50  0000 L CNN
-F 2 "JMG:HOLE_M2" H 6750 7600 50  0001 C CNN
+F 2 "Random-keyboard-parts:HOLE_M2" H 6750 7600 50  0001 C CNN
 F 3 "~" H 6750 7600 50  0001 C CNN
 	1    6750 7600
@@
 F 0 "JP4" V 3500 4700 50  0000 C CNN
 F 1 "GND" H 3500 4551 40  0001 C CNN
-F 2 "MYLIB:Jumper" H 3400 4700 60  0001 C CNN
+F 2 "Random-keyboard-parts:Jumper_Small" H 3400 4700 60  0001 C CNN
 F 3 "" H 3400 4700 60  0000 C CNN
 	1    3400 4700

Commit message: Update libs
Parts:
- D1, D10, D11, D12, D13, D14, D15, D16, D17, D18, D19, D2, D20, D21, D22, D23, D24, D25, D26, D27, D28, D29, D3, D30, D31, D32, D4, D5, D6, D7, D8, D9: footprint Random-keyboard-parts:D_SOD-123_dual_reversed -> cipulot_parts:D_SOD-123_dual_reversed
- H1, H2, H3, H4, H5, H6, H7, H8, H9: footprint Random-keyboard-parts:HOLE_M2_TH -> cipulot_parts:HOLE_M2_TH
- H10, H11, H12, H13: footprint Random-keyboard-parts:HOLE_M2 -> cipulot_parts:HOLE_M2
- J1: footprint Random-keyboard-parts:MJ-4PP-9 -> cipulot_parts:MJ-4PP-9
- JP10, JP11, JP4, JP5, JP7, JP8, JP9: footprint Random-keyboard-parts:Jumper_Small -> cipulot_parts:Jumper_Small; symbol random-keyboard-parts:Jumper_Small -> helixhschoc-rescue:Jumper_Small-random-keyboard-parts
- JP6: footprint Random-keyboard-parts:Jumper_Small -> cipulot_parts:Jumper_Small
- P1, P2: footprint Random-keyboard-parts:Pin_Small -> cipulot_parts:Pin_Small
- P3: footprint Random-keyboard-parts:OLED_Small -> cipulot_parts:OLED_Small
- P4: footprint Random-keyboard-parts:LED_Strip_Pad -> cipulot_parts:LED_Strip_Pad
- SW33: footprint Random-keyboard-parts:SW_3.5x6.0_TH -> cipulot_parts:SW_3.5x6.0_TH
- U1: footprint Arduino:Sparkfun_Pro_Micro_reversible -> cipulot_parts:Sparkfun_Pro_Micro_reversible
- U10, U11, U12, U13, U14, U15, U16, U17, U18, U19, U2, U20, U21, U22, U23, U24, U25, U26, U27, U28, U29, U3, U30, U31, U32, U33, U4, U5, U6, U7, U8, U9: footprint LED_WS_SK:SK6812MINI_rev -> cipulot_parts:SK6812MINI_rev

Commit message: Update PCB
Parts:
- SW1, SW10, SW11, SW12, SW13, SW14, SW15, SW16, SW17, SW18, SW19, SW2, SW20, SW21, SW22, SW23, SW24, SW25, SW26, SW27, SW28, SW29, SW3, SW30, SW31, SW32, SW4, SW5, SW6, SW7, SW8, SW9: footprint Keyswitches:Kailh_socket_PG1350_reversible_LEFT_nosilkangle -> cipulot_parts:Kailh_socket_PG1350_reversible_LEFT_nosilkangle
