File: PCB/kicad_6_hotswap_choc/helixhschoc.kicad_sch (KiCad schematic)
At the start: 126 parts, among them J1 MJ-4PP-9, P1 CONN_01X01, P2 CONN_01X01, P3 OLED, P4 LED, SW1 SW_PUSH, SW10 SW_PUSH, SW11 SW_PUSH, SW12 SW_PUSH, SW13 SW_PUSH, SW14 SW_PUSH, SW15 SW_PUSH, SW16 SW_PUSH, SW17 SW_PUSH, SW18 SW_PUSH, SW19 SW_PUSH, SW2 SW_PUSH, SW20 SW_PUSH, SW21 SW_PUSH, SW22 SW_PUSH, SW23 SW_PUSH, SW24 SW_PUSH, SW25 SW_PUSH, SW26 SW_PUSH, SW27 SW_PUSH, SW28 SW_PUSH, SW29 SW_PUSH, SW3 SW_PUSH, SW30 SW_PUSH, SW31 SW_PUSH, SW32 SW_PUSH, SW33 Reset, SW4 SW_PUSH, SW5 SW_PUSH, SW6 SW_PUSH, SW7 SW_PUSH, SW8 SW_PUSH, SW9 SW_PUSH, U1 ProMicro, U10 SK6812mini, U11 SK6812mini, U12 SK6812mini, U13 SK6812mini, U14 SK6812mini, U15 SK6812mini, U16 SK6812mini, U17 SK6812mini, U18 SK6812mini, U19 SK6812mini, U2 SK6812mini, U20 SK6812mini, U21 SK6812mini, U22 SK6812mini, U23 SK6812mini, U24 SK6812mini, U25 SK6812mini, U26 SK6812mini, U27 SK6812mini, U28 SK6812mini, U29 SK6812mini, U3 SK6812mini, U30 SK6812mini, U31 SK6812mini, U32 SK6812mini, U33 SK6812mini, U4 SK6812mini, U5 SK6812mini, U6 SK6812mini, U7 SK6812mini, U8 SK6812mini, U9 SK6812mini

Commit message: Update
Parts:
- D1: footprint cipulot_parts:D_SOD-123_dual_reversed -> cipulot_parts:D_SOD-123-Pretty
Changed lines of the file:
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@@
   (title_block
     (title "Helix HS Choc")
-    (date "2021-12-17")
+    (date "2021-12-27")
     (rev "v1.0")
     (comment 1 "Copyright © 2021 Cipulot")
@@
     (property "Reference" "D1" (id 0) (at 246.38 54.61 0))
     (property "Value" "D" (id 1) (at 251.46 54.61 0))
-    (property "Footprint" "cipulot_parts:D_SOD-123_dual_reversed" (id 2) (at 248.92 54.61 0)
+    (property "Footprint" "cipulot_parts:D_SOD-123-Pretty" (id 2) (at 248.92 54.61 0)
       (effects (font (size 1.27 1.27)) hide)
     )
@@
     )
     (path "/00000000-0000-0000-0000-00005986acfa"
-      (reference "D1") (unit 1) (value "D") (footprint "cipulot_parts:D_SOD-123_dual_reversed")
+      (reference "D1") (unit 1) (value "D") (footprint "cipulot_parts:D_SOD-123-Pretty")
     )
     (path "/00000000-0000-0000-0000-00005986ae36"
